Commit message: 03/12/2016 add odom_dev branch, to simulate the same input of gmapping, code modification: remove submap topic, point cloud topic and make map topic update 15 sec, more things to do later

File: cartographer_ros/cartographer_ros/urdf/backpack_2d.urdf (robot description, URDF)
Before this commit: robot cartographer_backpack_2d, 4 links, 3 joints
Links:
- removed link horizontal_laser_link
- removed link imu_link
- removed link vertical_laser_link
- link base_link: geometry visual cylinder length=0.4 radius=0.2
Joints:
- removed joint horizontal_laser_link_joint
- removed joint imu_link_joint
- removed joint vertical_laser_link_joint
